File: eagle/CiderPress.brd (EAGLE design)
At the start: 17.8 x 33 mm, 38 parts, among them Q1 8/16/20MHz, U1 ATMEGA328, U2 L7805CDT-TR, U3 BRM-2A18VERT, U4 NZT7053

Commit message: Work on Board
Parts:
- added JP11: (no value), SparkFun-Connectors:JST-4-PTH
- D1: value (none) -> 1N4001
Connections:
- net D2 renamed VALVE
- removed net A0: JP6.8, U1.23
- removed net A1: JP6.7, U1.24
- removed net A3: JP6.5, U1.26
- removed net D4: HIGH.2, JP7.6, R1.1, S2.1, S2.2, U1.2
- removed net D5: JP7.5, LOW.2, R3.1, S3.1, S3.2, U1.9
- removed net D6: JP7.4, U1.10
- removed net D9: JP10.3, JP7.1, U1.13
- new net GRN: JP10.1, JP6.7, U1.24
- new net IR: JP6.5, U1.26, U3.1
- new net RED: JP10.3, JP6.8, U1.23
- new net SSRX: JP11.1, JP7.2, U1.12
- new net SSTX: JP11.2, JP7.1, U1.13
- new net SWH: HIGH.2, JP7.3, R1.1, S2.1, S2.2, U1.11
- new net SWL: JP7.4, LOW.2, R3.1, S3.1, S3.2, U1.10
- net D10: no longer JP10.1
- net D3: no longer U3.1
- net ECHO: now also JP7.6, U1.2; no longer JP7.3, U1.11
- net GND: now also JP11.4
- net RAW: now also D1.C, JP9.2
- net TRIG: now also JP7.5, U1.9; no longer JP7.2, U1.12
- net VCC: now also JP11.3; no longer D1.C, JP9.2
Routing:
- net D9: track 12.4 -> 0.00 mm
- net D4: track 12.3 -> 0.00 mm, vias 1 -> 0
- net TRIG: track 9.97 -> 0.00 mm
- net ECHO: track 7.62 -> 0.00 mm
- net SWL: track 0.00 -> 5.71 mm
- net D6: track 5.71 -> 0.00 mm
- net IR: track 0.00 -> 5.06 mm
- net A3: track 5.06 -> 0.00 mm
- net A0: track 3.55 -> 0.00 mm
- net A1: track 3.31 -> 0.00 mm
- net D5: track 3.22 -> 0.00 mm
- net D3: track 12.0 -> 9.64 mm
- net GRN: track 0.00 -> 1.51 mm
- net RED: track 0.00 -> 1.30 mm
- net VALVE: track 9.45 -> 8.57 mm

Commit message: Place components
Parts:
- removed JP10: (no value), SparkFun-Connectors:JST-3-PTH
- removed JP11, JP12: (no value), SparkFun-Connectors:JST-4-PTH
- removed JP5, JP8: FIDUCIALUFIDUCIAL, SparkFun:MICRO-FIDUCIAL
- removed JP9: (no value), SparkFun-Connectors:JST-2-PTH
- removed U$1: LOGO-SFESK, SparkFun:SFE-LOGO-FLAME
- removed U$11: LOGO-SFENEW, SparkFun:SFE-NEW-WEBLOGO
- removed U$3: OSHW-LOGOS, SparkFun:OSHW-LOGO-S
- added 7SEG, DST: (no value), SparkFun-Connectors:JST-4-PTH
- added ISP_V13: (no value), SparkFun-Connectors:1X06
- added LEDS: (no value), SparkFun-Connectors:JST-3-PTH
- added SLD: (no value), SparkFun-Connectors:JST-2-PTH
- moved S3 123.3 mm to (16.5, 11.8)
- moved S2 123.0 mm to (15.6, 18.5), turned to 270 degrees
- moved R1 118.2 mm to (15.0, 23.9), turned to 180 degrees
- moved U3 115.2 mm to (33.7, 2.29)
- moved R3 113.1 mm to (16.9, 7.75)
- moved D1 111.1 mm to (14.0, 32.0), turned to 90 degrees
- moved JP4 100.9 mm to (37.0, 39.6), turned to 180 degrees
- moved U4 90.5 mm to (19.1, 31.2), turned to 180 degrees
- moved LOW 88.4 mm to (10.5, 12.6), turned to 90 degrees
- moved HIGH 87.4 mm to (10.5, 18.9), turned to 90 degrees
- moved U2 78.6 mm to (26.2, 32.9)
- moved JP2 28.1 mm to (39.9, 8.00)
- moved JP6 28.0 mm to (43.7, 36.1)
- moved JP3 26.1 mm to (39.2, 2.54)
- moved C19 24.9 mm to (38.0, 21.8), turned to 180 degrees
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Connections:
- net A4: now also U1.27
- net A5: now also U1.28
- net ECHO: now also DST.3; no longer JP12.3
- net GND: now also 7SEG.4, DST.4, ISP_V13.6, LEDS.2; no longer JP10.2, JP11.4, JP12.4
- net GRN: now also LEDS.1; no longer JP10.1
- net MISO: now also ISP_V13.3
- net MOSI: now also ISP_V13.2
- net N$6: now also SLD.1; no longer JP9.1
- net RAW: now also SLD.2; no longer JP9.2
- net RED: now also LEDS.3; no longer JP10.3
- net RESET: now also ISP_V13.1
- net SCK: now also ISP_V13.5
- net SSRX: now also 7SEG.1; no longer JP11.1
- net SSTX: now also 7SEG.2; no longer JP11.2
- net TRIG: now also DST.2; no longer JP12.2
- net VCC: now also 7SEG.3, DST.1, ISP_V13.4; no longer JP11.3, JP12.1
Routing:
- net VCC: track 48.5 -> 180.2 mm, vias 2 -> 11
- net SCK: track 9.94 -> 86.2 mm, vias 0 -> 4
- net MISO: track 19.7 -> 81.4 mm, vias 1 -> 4
- net RESET: track 63.7 -> 120.9 mm, vias 2 -> 4
- net RAW: track 0.00 -> 55.0 mm
- net MOSI: track 17.1 -> 69.7 mm, vias 1 -> 7
- net SWH: track 0.00 -> 38.6 mm, vias 0 -> 1
- net ECHO: track 0.00 -> 37.9 mm, vias 0 -> 1
- net VALVE: track 8.57 -> 46.3 mm, vias 1 -> 3
- net IR: track 5.06 -> 40.8 mm, vias 0 -> 2
- net TXO: track 25.8 -> 59.2 mm, vias 0 -> 3
- net D3: track 9.64 -> 39.6 mm, vias 1 -> 2
- net TRIG: track 0.00 -> 29.9 mm, vias 0 -> 1
- net SSTX: track 0.00 -> 26.4 mm, vias 0 -> 1
- net SSRX: track 0.00 -> 25.8 mm, vias 0 -> 1
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Other:
- board size 17.8 x 33 mm -> 45.7 x 43.8 mm
- board text added: "CiderPress V0"
- board text added: "DTR"
- board text added: "MISO"
- board text added: "MOSI"
- board text added: "Original Arduino Mini Design by Team Arduino Arduino Pro Mini Design by SparkFun Electronics Revised by Pete Lewis, CiderPress by Benjamin Guest"
- board text added: "SCK"
- board text removed: "10MHz"
- board text removed: "16MHz"
- board text removed: "20MHz"
- board text removed: "3.3V"
- board text removed: "5V"
- board text removed: "8MHz"
- board text removed: "Arduino Pro"
- board text removed: "Arduino Pro Mini"
- board text removed: "BLK"
- board text removed: "GRN"
- board text removed: "Mini"
- board text removed: "Original Arduino Mini Design by Team Arduino Arduino Pro Mini Design by SparkFun Electronics Revised by Pete Lewis"
- board text removed: "Reset"
- board text removed: "v14"
- board text removed: "www.arduino.cc"

Commit message: Update led resistor numbers
Parts:
- R11: value 10K -> 300
- R6: value 330 -> 300
Changed lines of the file:
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@@
 <?xml version="1.0" encoding="utf-8"?>
 <!DOCTYPE eagle SYSTEM "eagle.dtd">
-<eagle version="7.4.0">
+<eagle version="7.5.0">
 <drawing>
 <settings>
@@
 <attribute name="VALUE" x="22.2123" y="26.4033" size="0.8128" layer="27"/>
 </element>
-<element name="R11" library="adafruit" package="M0805" value="10K" x="32.893" y="22.225" smashed="yes" rot="R180">
+<element name="R11" library="adafruit" package="M0805" value="300" x="32.893" y="22.225" smashed="yes" rot="R180">
 <attribute name="VALUE" x="35.179" y="21.082" size="0.8128" layer="27" rot="R180"/>
 </element>
@@
 <attribute name="VALUE" x="15.5702" y="2.0447" size="0.8128" layer="27" rot="R90"/>
 </element>
-<element name="R6" library="adafruit" package="M0805" value="330" x="27.432" y="8.9662" smashed="yes" rot="R270">
+<element name="R6" library="adafruit" package="M0805" value="300" x="27.432" y="8.9662" smashed="yes" rot="R270">
 <attribute name="VALUE" x="29.4005" y="8.4333" size="0.8128" layer="27" rot="R90"/>
 </element>
