File: eagle/CiderPress.sch (EAGLE design)
At the start: 38 parts, among them Q1 8/16/20MHz, U1 ATMEGA328, U2 L7805CDT-TR, U3 BRM-2A18VERT, U4 NZT7053

Commit message: Work on Board
Parts:
- added JP11: (no value), SparkFun-Connectors:M04JST-PTH
- D1: value (none) -> 1N4001
Connections:
- net D2 renamed VALVE
- removed net A0: JP6.8, U1.PC0(ADC0)
- removed net A1: JP6.7, U1.PC1(ADC1)
- removed net A3: JP6.5, U1.PC3(ADC3)
- removed net D4: HIGH.2, JP7.6, R1.1, S2.1, U1.PD4(XCK/T0)
- removed net D5: JP7.5, LOW.2, R3.1, S3.1, U1.PD5(T1)
- removed net D6: JP7.4, U1.PD6(AIN0)
- removed net D9: JP10.3, JP7.1, U1.PB1(OC1A)
- new net GRN: JP10.1, JP6.7, U1.PC1(ADC1)
- new net IR: JP6.5, U1.PC3(ADC3), U3.OUT
- new net RED: JP10.3, JP6.8, U1.PC0(ADC0)
- new net SSRX: JP11.1, JP7.2, U1.PB0(ICP)
- new net SSTX: JP11.2, JP7.1, U1.PB1(OC1A)
- new net SWH: HIGH.2, JP7.3, R1.1, S2.1, U1.PD7(AIN1)
- new net SWL: JP7.4, LOW.2, R3.1, S3.1, U1.PD6(AIN0)
- net D10: no longer JP10.1
- net D3: no longer U3.OUT
- net ECHO: now also JP7.6, U1.PD4(XCK/T0); no longer JP7.3, U1.PD7(AIN1)
- net GND: now also JP11.4
- net RAW: now also D1.C, JP9.2
- net TRIG: now also JP7.5, U1.PD5(T1); no longer JP7.2, U1.PB0(ICP)
- net VCC: now also JP11.3; no longer D1.C, JP9.2
Other:
- note added: "4x7 Segment Display"

Commit message: Place components
Parts:
- removed JP5, JP8: FIDUCIALUFIDUCIAL, SparkFun:FIDUCIALUFIDUCIAL
- removed U$1: LOGO-SFESK, SparkFun:LOGO-SFESK
- removed U$11: LOGO-SFENEW, SparkFun:LOGO-SFENEW
- removed U$3: OSHW-LOGOS, SparkFun:OSHW-LOGOS
- added ISP_V13: (no value), SparkFun-Connectors:M06SIP
- renumbered JP10 to LEDS, JP11 to 7SEG, JP12 to DST, JP9 to SLD
Connections:
- net A4: now also U1.PC4(ADC4/SDA)
- net A5: now also U1.PC5(ADC5/SCL)
- net GND: now also ISP_V13.6
- net MISO: now also ISP_V13.3
- net MOSI: now also ISP_V13.2
- net RESET: now also ISP_V13.1
- net SCK: now also ISP_V13.5
- net VCC: now also ISP_V13.4

Commit message: Update led resistor numbers
Parts:
- R11: value 10K -> 300
- R6: value 330 -> 300
Changed lines of the file:
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@@
 <?xml version="1.0" encoding="utf-8"?>
 <!DOCTYPE eagle SYSTEM "eagle.dtd">
-<eagle version="7.4.0">
+<eagle version="7.5.0">
 <drawing>
 <settings>
@@
 <part name="FRAME1" library="SparkFun-Aesthetics" deviceset="FRAME-LETTER" device=""/>
 <part name="GND26" library="SparkFun" deviceset="GND" device=""/>
-<part name="R11" library="adafruit" deviceset="R-US_" device="M0805" value="10K"/>
+<part name="R11" library="adafruit" deviceset="R-US_" device="M0805" value="300"/>
 <part name="LED1" library="adafruit" deviceset="LED" device="CHIPLED_0805" value="Red"/>
 <part name="GND28" library="SparkFun" deviceset="GND" device=""/>
@@
 <part name="C1" library="adafruit" deviceset="C-US" device="C0805" value="0.1uF"/>
 <part name="GND7" library="SparkFun" deviceset="GND" device=""/>
-<part name="R6" library="adafruit" deviceset="R-US_" device="M0805" value="330"/>
+<part name="R6" library="adafruit" deviceset="R-US_" device="M0805" value="300"/>
 <part name="D3" library="adafruit" deviceset="LED" device="CHIPLED_0805" value="Green"/>
 <part name="GND8" library="SparkFun" deviceset="GND" device=""/>
